Commit message: changes

File: ada_description/robots/mico.urdf (robot description, URDF)
Before this commit: robot ADA, 16 links, 15 joints
Links:
- removed link Camera_Collision_Frame
- removed link Camera_Depth_Frame
- removed link Camera_RGB_Frame
Joints:
- removed joint Camera_Collision_Joint
- removed joint Camera_Depth_Joint
- removed joint Camera_Joint
